File: touch_keypad.kicad_sch (KiCad schematic)
At the start: 42 parts, among them J1 USB_B_Micro, J5 Conn_01x04_Female, SW1 SW_Push, SW10 SW_Push, SW11 SW_Push, SW12 SW_Push, SW13 SW_Push, SW14 SW_Push, SW15 SW_Push, SW16 SW_Push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

Commit message: output
Parts:
- removed Y1: Crystal, Crystal:Crystal_HC18-U_Vertical, symbol Device:Crystal
- added C? (x2): 47n, Capacitor_SMD:C_0603_1608Metric_Pad1.05x0.95mm_HandSolder, symbol Device:C
- added R? (x6): R, Resistor_SMD:R_0603_1608Metric_Pad1.05x0.95mm_HandSolder, symbol Device:R
- added Y1: Crystal_GND24, Crystal:Crystal_SMD_3225-4Pin_3.2x2.5mm, symbol Device:Crystal_GND24
Connections:
- net +3V3: now also C7.1
- net Button1: now also U2.6 (PA0), R?.1; no longer SW10.1, SW15.1, SW5.1, SW7.1, U2.7 (PA1)
- net Button2: now also U2.7 (PA1), R?.1; no longer SW12.1, SW16.1, SW3.1, SW8.1, U2.8 (PA2)
- net Button3: now also U2.8 (PA2), R?.1; no longer SW13.1, SW17.1, SW4.1, SW9.1, U2.9 (PA3)
- net Button4: now also R?.1; no longer SW6.1, SW7.2, SW8.2, SW9.2
- net Button5: now also R?.1; no longer SW10.2, SW11.1, SW12.2, SW13.2
- net Button6: now also R?.1; no longer SW14.1, SW15.2, SW16.2, SW17.2
- net GND: now also J1.6 (Shield), C?.2, C?.2
- net Sampling_cap1: now also U2.9 (PA3), C?.1; no longer U2.6 (PA0)
- net Sampling_cap2: now also C?.1
- net at C1.1: now also Y1.2; no longer U2.2 (PF0)
- net at C2.1: now also Y1.4; no longer U2.3 (PF1)
- new net: U2.2 (PF0), Y1.1
- new net: U2.3 (PF1), Y1.3
- new net: R?.2, SW10.1, SW15.1, SW5.1, SW7.1
- new net: R?.2, SW12.1, SW16.1, SW3.1, SW8.1
- new net: R?.2, SW13.1, SW17.1, SW4.1, SW9.1
- new net: R?.2, SW6.1, SW7.2, SW8.2, SW9.2
- new net: R?.2, SW10.2, SW11.1, SW12.2, SW13.2
- new net: R?.2, SW14.1, SW15.2, SW16.2, SW17.2
Other:
- moved on the sheet: C1, C2
